Commit message: Caracterizacion VICON

File: src/charlie_description/vicon_urdf/robot.urdf.xacro (robot description, xacro)
@@ -46,5 +46,5 @@
         <parent link="base_link"/>
         <child link="lidar_link"/>
-        <origin xyz="0 0 0.2" rpy="0 0 0"/>
+        <origin xyz="0 0 0.2" rpy="0 0 3.14"/>
     </joint>
 </robot>
