Commit message: Ackerman se mueve raro - Modificación EKF

File: src/charlie_description/ackermann_urdf/robot_core.xacro (robot description, xacro)
@@ -56,10 +56,10 @@
                 <material name="${p_color}"/>
             </visual>
-            <collision>
+            <!-- <collision>
                 <origin xyz="0 0 0"/>
                 <geometry>
                     <cylinder radius="${p_radius}" length="${p_length}"/>
                 </geometry>
-            </collision>
+            </collision> -->
             <xacro:inertial_cylinder mass="${p_mass}" length="${p_length}" radius="${p_radius}">
                 <origin xyz="0 0 0" rpy="0 0 0"/>

File: src/charlie_description/ackermann_urdf/ros2_control.xacro (robot description, xacro)
@@ -39,4 +39,12 @@
       <state_interface name="position"/>
     </joint>
+    <joint name="left_front_wheel_joint">
+      <state_interface name="position"/>
+      <state_interface name="velocity"/>
+    </joint>
+    <joint name="right_front_wheel_joint">
+      <state_interface name="position"/>
+      <state_interface name="velocity"/>
+    </joint>
   </ros2_control>
   <gazebo>

Commit message: Esto no servía XD

File: src/charlie_description/ackermann_urdf/robot_core.xacro (robot description, xacro)
@@ -46,4 +46,7 @@
             </xacro:inertial_cylinder>
         </link>
+        <gazebo reference="${p_name}">
+            <mu1>1.5</mu1> <mu2>1.5</mu2> <kp>10000000.0</kp> <kd>1.0</kd> <minDepth>0.001</minDepth>
+        </gazebo>
     </xacro:macro>
     <xacro:macro name="steering_macro" params="p_name p_radius p_length p_color p_mass">
@@ -142,5 +145,5 @@
         <child link="left_steering_link"/>
         <origin xyz="${lx/2 - offset} ${ly/2+steering_r} -${lz}" rpy="0 0 0"/> <!-- For wheelbase --> <!-- For steering & traction track -->
-        <axis xyz="0 0 1"/>
+        <axis xyz="0 0 -1"/>
         <limit lower="-${pi/4}" upper="${pi/4}" effort="5.0" velocity="1.0"/>
         <dynamics damping="0.5" friction="0.0"/>
@@ -150,5 +153,5 @@
         <child link="right_steering_link"/>
         <origin xyz="${lx/2 - offset} -${ly/2 + steering_r} -${lz}" rpy="0 0 0"/> <!-- For steering & traction track -->
-        <axis xyz="0 0 1"/>
+        <axis xyz="0 0 -1"/>
         <limit lower="-${pi/4}" upper="${pi/4}" effort="5.0" velocity="1.0"/>
         <dynamics damping="0.5" friction="0.0"/>

Commit message: Simulation ok

File: src/charlie_description/ackermann_urdf/robot_core.xacro (robot description, xacro)
@@ -3,5 +3,4 @@
     <!-- Include macros -->
     <xacro:include filename="$(find charlie_description)/macros/inertial_macros.xacro"/>
-    <!--Measurements-->
     <xacro:property name="rad_w" value="0.053"/>
     <xacro:property name="le_w" value="0.045"/>
@@ -18,6 +17,14 @@
     <xacro:property name="imu_ly" value="0.03"/>
     <xacro:property name="imu_lz" value="0.01"/>
+    <xacro:macro name="phantom_steer_link" params="p_name">
+        <link name="${p_name}">
+            <inertial>
+                <mass value="0.05"/>
+                <origin xyz="0 0 0" rpy="0 0 0"/>
+                <inertia ixx="0.00001" ixy="0" ixz="0" iyy="0.00001" iyz="0" izz="0.00001"/>
+            </inertial>
+        </link>
+    </xacro:macro>
     <xacro:macro name="wheel_macro" params="p_name p_radius p_width">
-    <!-- ... -->
         <link name="${p_name}">
             <visual>
@@ -38,5 +45,4 @@
     </xacro:macro>
     <xacro:macro name="barras" params="p_name p_x p_y p_z">
-    <!-- ... -->
         <link name="${p_name}">
             <visual>
@@ -59,5 +65,4 @@
     </xacro:macro>
     <xacro:macro name="barra_horizontal" params="p_name p_x p_y p_z origin">
-    <!-- ... -->
         <link name="${p_name}">
             <visual>
@@ -79,7 +84,5 @@
         </link>
     </xacro:macro>
-    <!-- Example link -->
-    <link name="base_link">
-    </link>
+    <link name="base_link"></link>
     <joint name="base_link_joint" type="fixed">
         <parent link="base_link"/>
@@ -128,40 +131,32 @@
         </xacro:inertial_box>
     </link>
-    <!--Pata trasera derecha-->
     <joint name="chassis_verticalbar_1" type="fixed">
         <parent link="chassis"/>
         <child link="barra_vertical_tr_link"/>
+        <origin xyz="${-0.257/2} ${ly/3} ${bscz+0.008}"/>
+    </joint>
+    <xacro:barras p_name="barra_vertical_tr_link" p_x="${bscx}" p_y="${bscy}" p_z="${bscz}"/>
+    <joint name="chassis_verticalbar_2" type="fixed">
+        <parent link="chassis"/>
+        <child link="barra_vertical_tr_l_link"/>
+        <origin xyz="${-0.257/2} ${-ly/3} ${bscz+0.008}"/>
+    </joint>
+    <xacro:barras p_name="barra_vertical_tr_l_link" p_x="${bscx}" p_y="${bscy}" p_z="${bscz}"/>
+    <joint name="chassis_verticalbar_3" type="fixed">
+        <parent link="chassis"/>
+        <child link="barra_vertical_de_link"/>
         <origin xyz="${0.257/2} ${ly/3} ${bscz+0.008}"/>
     </joint>
-    <xacro:barras p_name="barra_vertical_tr_link" p_x="${bscx}" p_y="${bscy}" p_z="${bscz}"/>
-    <!--Pata trasera izquierda-->
-    <joint name="chassis_verticalbar_2" type="fixed">
-        <parent link="chassis"/>
-        <child link="barra_vertical_tr_l_link"/>
+    <xacro:barras p_name="barra_vertical_de_link" p_x="${bscx}" p_y="${bscy}" p_z="${bscz}"/>
+    <joint name="chassis_verticalbar_4" type="fixed">
+        <parent link="chassis"/>
+        <child link="barra_vertical_de_l_link"/>
         <origin xyz="${0.257/2} ${-ly/3} ${bscz+0.008}"/>
     </joint>
-    <xacro:barras p_name="barra_vertical_tr_l_link" p_x="${bscx}" p_y="${bscy}" p_z="${bscz}"/>
-    <!--Pata delantera derecha-->
-    <joint name="chassis_verticalbar_3" type="fixed">
-        <parent link="chassis"/>
-        <child link="barra_vertical_de_link"/>
-        <origin xyz="${-0.257/2} ${ly/3} ${bscz+0.008}"/>
-    </joint>
-    <xacro:barras p_name="barra_vertical_de_link" p_x="${bscx}" p_y="${bscy}" p_z="${bscz}"/>
-    <!--Pata trasera izquierda-->
-    <joint name="chassis_verticalbar_4" type="fixed">
-        <parent link="chassis"/>
-        <child link="barra_vertical_de_l_link"/>
-        <origin xyz="${-0.257/2} ${-ly/3} ${bscz+0.008}"/>
-    </joint>
     <xacro:barras p_name="barra_vertical_de_l_link" p_x="${bscx}" p_y="${bscy}" p_z="${bscz}"/>
-    <!--Barra trasera derecha-->
-    <joint name="chassis_horizontalbar_1" type="revolute">
+    <joint name="chassis_horizontalbar_tr" type="fixed">
         <parent link="chassis"/>
         <child link="barra_horizontal_tr_link"/>
-        <origin xyz="${0.257/2} 0.035  ${-(lz+bhz)/2}" rpy="0 0 0"/>
-        <axis xyz="0 0 1"/>
-        <limit effort="1" lower="-${pi/4}" upper="${pi/4}" velocity="1"/>
-        <dynamics damping="0.2" friction="0"/>
+        <origin xyz="${-0.257/2} 0.035  ${-(lz+bhz)/2}" rpy="0 0 0"/>
     </joint>
     <xacro:barra_horizontal p_name="barra_horizontal_tr_link" p_x="${bhx}" p_y="${bhy}" p_z="${bhz}" origin="${0.0175}"/>
@@ -174,12 +169,8 @@
     </joint>
     <xacro:wheel_macro p_name="rightb_wheel" p_radius="${rad_w}" p_width="${le_w}"/>
-      <!--Barra trasera izquierda-->
-    <joint name="chassis_horizontalbar_2" type="revolute">
+    <joint name="chassis_horizontalbar_ti" type="fixed">
         <parent link="chassis"/>
         <child link="barra_horizontal_ti_link"/>
-        <origin xyz="${0.257/2} -0.035  ${-(lz+bhz)/2}" rpy="0 0 0"/>
-        <axis xyz="0 0 1"/>
-        <limit effort="1" lower="-${pi/4}" upper="${pi/4}" velocity="1"/>
-        <dynamics damping="0.2" friction="0"/>
+        <origin xyz="${-0.257/2} -0.035  ${-(lz+bhz)/2}" rpy="0 0 0"/>
     </joint>
     <xacro:barra_horizontal p_name="barra_horizontal_ti_link" p_x="${bhx}" p_y="${bhy}" p_z="${bhz}" origin="${-0.0175}"/>
@@ -192,36 +183,46 @@
     </joint>
     <xacro:wheel_macro p_name="leftb_wheel" p_radius="${rad_w}" p_width="${le_w}"/>
-    <!--Barra delantera derecha-->
-    <joint name="chassis_horizontalbar_3" type="revolute">
+    <joint name="chassis_horizontalbar_fr" type="fixed">
         <parent link="chassis"/>
         <child link="barra_horizontal_fr_link"/>
-        <origin xyz="${-0.257/2} 0.035  ${-(lz+bhz)/2}" rpy="0 0 0"/>
-        <axis xyz="0 0 1"/>
-        <limit effort="1" lower="-${pi/4}" upper="${pi/4}" velocity="1"/>
-        <dynamics damping="0.2" friction="0"/>
+        <origin xyz="${0.257/2} 0.035  ${-(lz+bhz)/2}" rpy="0 0 0"/>
     </joint>
     <xacro:barra_horizontal p_name="barra_horizontal_fr_link" p_x="${bhx}" p_y="${bhy}" p_z="${bhz}" origin="${0.0175}"/>
+    <xacro:phantom_steer_link p_name="right_steering_link"/>
+    <joint name="right_steering_joint" type="revolute">
+        <parent link="barra_horizontal_fr_link"/>
+        <child link="right_steering_link"/>
+        <origin xyz="0 ${0.055+le_w/2} 0" rpy="0 0 0"/>
+        <axis xyz="0 0 1"/>
+        <limit effort="5.0" lower="-${pi/4}" upper="${pi/4}" velocity="5.0"/>
+        <dynamics damping="0.2" friction="0.1"/>
+    </joint>
     <joint name="rightf_wheel_joint" type="continuous">
-        <parent link="barra_horizontal_fr_link"/>
+        <parent link="right_steering_link"/>
         <child link="rightf_wheel"/>
-        <origin xyz="0 ${0.055+le_w/2} 0" rpy="-${pi/2} 0 0"/>
+        <origin xyz="0 0 0" rpy="-${pi/2} 0 0"/>
         <axis xyz="0 0 1"/>
         <dynamics damping="0.2" friction="0.0"/>
     </joint>
     <xacro:wheel_macro p_name="rightf_wheel" p_radius="${rad_w}" p_width="${le_w}"/>
-    <!--Barra delantera izquierda-->
-    <joint name="chassis_horizontalbar_4" type="revolute">
+    <joint name="chassis_horizontalbar_fi" type="fixed">
         <parent link="chassis"/>
         <child link="barra_horizontal_fi_link"/>
-        <origin xyz="${-0.257/2} -0.035  ${-(lz+bhz)/2}" rpy="0 0 0"/>
-        <axis xyz="0 0 1"/>
-        <limit effort="1" lower="-${pi/4}" upper="${pi/4}" velocity="1"/>
-        <dynamics damping="0.2" friction="0"/>
+        <origin xyz="${0.257/2} -0.035  ${-(lz+bhz)/2}" rpy="0 0 0"/>
     </joint>
     <xacro:barra_horizontal p_name="barra_horizontal_fi_link" p_x="${bhx}" p_y="${bhy}" p_z="${bhz}" origin="${-0.0175}"/>
+    <xacro:phantom_steer_link p_name="left_steering_link"/>
+    <joint name="left_steering_joint" type="revolute">
+        <parent link="barra_horizontal_fi_link"/>
+        <child link="left_steering_link"/>
+        <origin xyz="0 ${-(0.055+le_w/2)} 0" rpy="0 0 0"/>
+        <axis xyz="0 0 1"/>
+        <limit effort="5.0" lower="-${pi/4}" upper="${pi/4}" velocity="5.0"/>
+        <dynamics damping="0.2" friction="0.1"/>
+    </joint>
     <joint name="leftf_wheel_joint" type="continuous">
-        <parent link="barra_horizontal_fi_link"/>
+        <parent link="left_steering_link"/>
         <child link="leftf_wheel"/>
-        <origin xyz="0 ${-(0.055+le_w/2)} 0" rpy="-${pi/2} 0 0"/>
+        <origin xyz="0 0 0" rpy="-${pi/2} 0 0"/>
         <axis xyz="0 0 1"/>
         <dynamics damping="0.2" friction="0.0"/>

File: src/charlie_description/ackermann_urdf/ros2_control.xacro (robot description, xacro)
@@ -6,16 +6,16 @@
     </hardware>
     <!-- Steering joints (front) -->
-    <joint name="chassis_horizontalbar_3">
+    <joint name="left_steering_joint">
       <command_interface name="position">
-        <param name="min">-0.7</param>
-        <param name="max">0.7</param>
+        <param name="min">-0.785</param>
+        <param name="max">0.785</param>
       </command_interface>
       <state_interface name="position"/>
       <state_interface name="velocity"/>
     </joint>
-    <joint name="chassis_horizontalbar_4">
+    <joint name="right_steering_joint">
       <command_interface name="position">
-        <param name="min">-0.7</param>
-        <param name="max">0.7</param>
+        <param name="min">-0.785</param>
+        <param name="max">0.785</param>
       </command_interface>
       <state_interface name="position"/>

Commit message: Funciona mejor (?)

File: src/charlie_description/ackermann_urdf/robot_core.xacro (robot description, xacro)
@@ -46,6 +46,6 @@
             <mu1>1.0</mu1>
             <mu2>0.5</mu2>
-            <kp>10000000.0</kp>
-            <kd>1.0</kd>
+            <kp>100000.0</kp>
+            <kd>100.0</kd>
             <minDepth>0.001</minDepth>
             <maxVel>0.1</maxVel>
@@ -203,5 +203,5 @@
         <origin xyz="0 ${0.055+le_w/2} 0" rpy="0 0 0"/>
         <axis xyz="0 0 1"/>
-        <limit effort="5.0" lower="-${pi/4}" upper="${pi/4}" velocity="5.0"/>
+        <limit effort="500.0" lower="-${pi/4}" upper="${pi/4}" velocity="5.0"/>
         <dynamics damping="0.2" friction="0.1"/>
     </joint>
@@ -226,5 +226,5 @@
         <origin xyz="0 ${-(0.055+le_w/2)} 0" rpy="0 0 0"/>
         <axis xyz="0 0 1"/>
-        <limit effort="5.0" lower="-${pi/4}" upper="${pi/4}" velocity="5.0"/>
+        <limit effort="500.0" lower="-${pi/4}" upper="${pi/4}" velocity="5.0"/>
         <dynamics damping="0.2" friction="0.1"/>
     </joint>
