Commit message: Rotación de IMU

File: src/charlie_description/sensors/imu_a.xacro (robot description, xacro)
@@ -22,5 +22,5 @@
         <parent link="chassis"/>
         <child link="imu_link"/>
-        <origin xyz="${0.06217} ${-0.025} ${lz/2 + imu_lz/2+0.036}" rpy="0 0 0"/>
+        <origin xyz="${0.06217} ${-0.025} ${lz/2 + imu_lz/2+0.036}" rpy="3.14159 0 0"/>
     </joint>
     <gazebo reference="imu_link">
