Commit message: Cambiios varios para que se mueva en rviz con el modelo de verdad

File: src/charlie_description/sensors/lidar_a1.xacro (robot description, xacro)
@@ -21,5 +21,5 @@
         <parent link="chassis"/>
         <child link="lidar_link"/>
-        <origin xyz="0 0 ${(lz+le_w/2)+0.016}" rpy="0 0 0"/>
+        <origin xyz="0 0 ${(lz+le_w/2)+0.016}" rpy="0 0 3.1416"/>
     </joint>
     <gazebo reference="lidar_link">
